File: pwr.kicad_sch (KiCad schematic)
At the start: 12 parts

Commit message: Schematic
Parts:
- removed C? (x3): .1u, Capacitor_SMD:C_0805_2012Metric_Pad1.18x1.45mm_HandSolder, symbol Device:C
- removed C? (x3): 2.2u, Capacitor_SMD:C_0805_2012Metric_Pad1.18x1.45mm_HandSolder, symbol Device:C
- removed L?: 10u, Inductor_SMD:L_TDK_VLS6045EX_VLS6045AF, symbol Device:L
- removed R?: 68k, Resistor_SMD:R_0805_2012Metric_Pad1.20x1.40mm_HandSolder, symbol Device:R
- removed R?: 10k, Resistor_SMD:R_0805_2012Metric_Pad1.20x1.40mm_HandSolder, symbol Device:R
- removed R?: 12k, Resistor_SMD:R_0805_2012Metric_Pad1.20x1.40mm_HandSolder, symbol Device:R
- removed U?: MIC5365-3.0, Package_TO_SOT_SMD:SOT-353_SC-70-5, symbol Regulator_Linear:MIC5365-3.3YC5
- removed U?: AP63200WU, Package_TO_SOT_SMD:TSOT-23-6, symbol Regulator_Switching:AP63200WU
Other:
- note removed: "6V Switching supply"
- note removed: "6V, 2A(max) Out"
- note removed: "VLS6045EX-100M"
