File: osci.kicad_sch (KiCad schematic)
At the start: 14 parts

Commit message: Schematic
Parts:
- removed C? (x2): .1u, symbol Device:C
- removed U? (x2): TL071, Package_SO:SOIC-8_3.9x4.9mm_P1.27mm, symbol Amplifier_Operational:TL071
- added C? (x2): .1u, symbol Device:C
- added R? (x2): 10k, symbol Device:R
- added U? (x4): LM324, symbol Amplifier_Operational:LM324
Connections:
- net +2V5: now also C?.1, R?.1, R?.2
- net +5V: now also R?.1
- net GND: now also C?.2, C?.2, R?.2, U?.11 (V-)
- net Pitch Antenna: now also U?.3 (+)
- net Pitch Frequency: now also U?.1
- net Volume Antenna: now also U?.5 (+)
- net Volume Frequency: now also U?.7
- net at R?.2: now also U?.2 (-)
- net at R?.2: now also U?.6 (-)
- new net: C?.1, U?.4 (V+)
Other:
- note added: "Vcc/2 Not necessarily 2.5V"
- moved on the sheet: C?, R?

Commit message: Schematics
Parts:
- removed C? (x4): .1u, symbol Device:C
- removed R? (x2): 10k, symbol Device:R
- removed R? (x2): 1M, symbol Device:R
- removed R? (x6): 100k, symbol Device:R
- removed U? (x4): LM324, symbol Amplifier_Operational:LM324
- added C? (x2): .1u, symbol Device:C
- added R? (x2): 1K, symbol Device:R
- added R? (x4): 1Meg, symbol Device:R
- added U? (x2): NE555P, Package_DIP:DIP-8_W7.62mm, symbol Timer:NE555P
Connections:
- net +5V: now also C?.1, C?.1, R?.1, R?.1, R?.1, R?.1, U?.4 (R), U?.4 (R), U?.7 (DIS), U?.7 (DIS), U?.8 (VCC), U?.8 (VCC)
- net GND: now also C?.2, C?.2, U?.1 (GND), U?.1 (GND)
- net Pitch Antenna: now also R?.2
- net Pitch Frequency: now also R?.2, U?.3 (Q)
- net Volume Antenna: now also R?.2
- net Volume Frequency: now also R?.2, U?.3 (Q)
- new net: R?.1, R?.2, U?.2 (TR), U?.6 (THR) (x2)
Other:
- note removed: "Vcc/2 Not necessarily 2.5V"

Commit message: PCB
Parts:
- removed C?: .1u, symbol Device:C
- removed R?: 1K, symbol Device:R
- removed R? (x2): 1Meg, symbol Device:R
- removed U?: NE555P, Package_DIP:DIP-8_W7.62mm, symbol Timer:NE555P
- added C13: .1u, Capacitor_THT:C_Rect_L4.0mm_W2.5mm_P2.50mm, symbol Device:C
- added R11: 1K, Resistor_THT:R_Axial_DIN0207_L6.3mm_D2.5mm_P10.16mm_Horizontal, symbol Device:R
- added R14, R15: 1Meg, Resistor_THT:R_Axial_DIN0207_L6.3mm_D2.5mm_P10.16mm_Horizontal, symbol Device:R
- added U4: NE555P, Package_DIP:DIP-8_W7.62mm, symbol Timer:NE555P
- C12: renamed from C?; footprint (none) -> Capacitor_THT:C_Rect_L4.0mm_W2.5mm_P2.50mm
- R10, R12, R13: renamed from R?; footprint (none) -> Resistor_THT:R_Axial_DIN0207_L6.3mm_D2.5mm_P10.16mm_Horizontal
- gave numbers to parts that had none: 1
Connections:
- net +5V: now also C13.1, R11.1, R14.1, U4.4 (R), U4.8 (VCC); no longer U3.7 (DIS)
- net GND: now also C13.2, U4.1 (GND)
- net Pitch Antenna: now also U3.2 (TR), U3.6 (THR)
- net Volume Antenna: now also R15.2, U4.2 (TR), U4.6 (THR)
- net Volume Frequency: now also R11.2, U4.3 (Q)
- net at R12.2, R13.1: now also U3.7 (DIS); no longer U3.2 (TR), U3.6 (THR)
- new net: R14.2, R15.1, U4.7 (DIS)
Other:
- moved on the sheet: R12, R13
