File: digital.kicad_sch (KiCad schematic)
At the start: 6 parts

Commit message: Schematics
Connections:
- net Calibrate Button: now also U?.7 (PA0); no longer U?.9 (PA2)
- net Sine LED: now also U?.18 (PA8); no longer U?.10 (PA3)
- net Volume Frequency: now also U?.9 (PA2); no longer U?.7 (PA0)
- new net Pitch Set: U?.10 (PA3)
Changed lines of the file:
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@@
   (junction (at 153.67 48.26) (diameter 0) (color 0 0 0 0)
+  )
+  (wire (pts (xy 121.92 82.55) (xy 135.89 82.55))
+    (stroke (width 0) (type default) (color 0 0 0 0))
   )
   (wire (pts (xy 120.65 119.38) (xy 120.65 123.19))
@@
     (stroke (width 0) (type default) (color 0 0 0 0))
   )
-  (wire (pts (xy 121.92 82.55) (xy 135.89 82.55))
+  (wire (pts (xy 121.92 85.09) (xy 135.89 85.09))
     (stroke (width 0) (type default) (color 0 0 0 0))
   )
-  (wire (pts (xy 121.92 85.09) (xy 135.89 85.09))
+  (wire (pts (xy 121.92 95.25) (xy 135.89 95.25))
     (stroke (width 0) (type default) (color 0 0 0 0))
   )
@@
     (effects (font (size 1.27 1.27)) (justify right))
   )
-  (hierarchical_label "Sine LED" (shape output) (at 121.92 82.55 180)
+  (hierarchical_label "Sine LED" (shape output) (at 121.92 95.25 180)
     (effects (font (size 1.27 1.27)) (justify right))
   )
-  (hierarchical_label "Volume Frequency" (shape input) (at 121.92 74.93 180)
+  (hierarchical_label "Volume Frequency" (shape input) (at 121.92 80.01 180)
     (effects (font (size 1.27 1.27)) (justify right))
   )
-  (hierarchical_label "Calibrate Button" (shape input) (at 121.92 80.01 180)
+  (hierarchical_label "Calibrate Button" (shape input) (at 121.92 74.93 180)
     (effects (font (size 1.27 1.27)) (justify right))
   )
@@
     (effects (font (size 1.27 1.27)) (justify right))
   )
+  (hierarchical_label "Pitch Set" (shape input) (at 121.92 82.55 180)
+    (effects (font (size 1.27 1.27)) (justify right))
+  )

Commit message: PCB
Parts:
- added SWD1: Conn_ARM_JTAG_SWD_10, Connector_PinHeader_1.27mm:PinHeader_2x05_P1.27mm_Vertical, symbol Connector:Conn_ARM_JTAG_SWD_10
- C14: renamed from C?; footprint (none) -> Capacitor_THT:C_Rect_L4.0mm_W2.5mm_P2.50mm
- JP1, JP2: renamed from JP?; footprint (none) -> Jumper:SolderJumper-2_P1.3mm_Open_TrianglePad1.0x1.5mm
- R16, R17: renamed from R?; footprint (none) -> Resistor_THT:R_Axial_DIN0207_L6.3mm_D2.5mm_P10.16mm_Horizontal
- gave numbers to parts that had none: 1
Connections:
- net +3V0: now also SWD1.1 (VTref)
- net GND: now also SWD1.3 (GND), SWD1.5 (GND)
- net swclk: now reaches JP1.2 (B), R16.1, U5.25 (PA14/BOOT0)
- net swclk: now also SWD1.4 (SWDCLK/TCK)
- net RST: now reaches JP2.1 (A), R17.2, U5.6 (~{RST}/PF2)
- net RST: now also SWD1.10 (~{RESET})
- net UART TX: now reaches U5.19 (PA9)
- net UART RX: now reaches U5.21 (PA10)
- net swdio: now reaches U5.24 (PA13)
- net swdio: now also SWD1.2 (SWDIO/TMS)
- no-connect marks 0 -> 3

Commit message: Update
Parts:
- SWD1: PN (none) -> 20021111-00010T1LF
Changed lines of the file:
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@@
+      (effects (font (size 1.27 1.27)) hide)
+    )
+    (property "PN" "20021111-00010T1LF" (id 4) (at 66.04 165.1 0)
       (effects (font (size 1.27 1.27)) hide)
     )
