File: tda2822 board/tda2822 board.kicad_sch (KiCad schematic)
At the start: 14 parts, among them J1 Conn_01x02_Female, J2 Conn_01x02_Female, J3 Conn_01x02_Female, U1 TDA2822

Commit message: Antenna mounts
Parts:
- removed C1: 100u, Capacitor_THT:CP_Radial_D5.0mm_P2.50mm, symbol Device:C_Polarized
Changed lines of the file:
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@@
 (kicad_sch (version 20211123) (generator eeschema)
   (paper "A4")
-  (junction (at 36.83 38.1) (diameter 0) (color 0 0 0 0)
-  )
-  (junction (at 36.83 30.48) (diameter 0) (color 0 0 0 0)
-  )
   (junction (at 115.57 140.97) (diameter 0) (color 0 0 0 0)
   )
@@
   (junction (at 69.85 29.21) (diameter 0) (color 0 0 0 0)
   )
-  (wire (pts (xy 36.83 27.94) (xy 36.83 30.48))
-    (stroke (width 0) (type default) (color 0 0 0 0))
-  )
-  (wire (pts (xy 36.83 38.1) (xy 36.83 44.45))
+  (wire (pts (xy 36.83 27.94) (xy 36.83 31.75))
+    (stroke (width 0) (type default) (color 0 0 0 0))
+  )
+  (wire (pts (xy 36.83 34.29) (xy 36.83 44.45))
     (stroke (width 0) (type default) (color 0 0 0 0))
   )
@@
     (stroke (width 0) (type default) (color 0 0 0 0))
   )
-  (wire (pts (xy 36.83 30.48) (xy 45.72 30.48))
-    (stroke (width 0) (type default) (color 0 0 0 0))
-  )
   (wire (pts (xy 100.33 77.47) (xy 100.33 78.74))
     (stroke (width 0) (type default) (color 0 0 0 0))
@@
     (stroke (width 0) (type default) (color 0 0 0 0))
   )
-  (wire (pts (xy 45.72 38.1) (xy 36.83 38.1))
-    (stroke (width 0) (type default) (color 0 0 0 0))
-  )
   (wire (pts (xy 147.32 81.28) (xy 151.13 81.28))
     (stroke (width 0) (type default) (color 0 0 0 0))
@@
     (stroke (width 0) (type default) (color 0 0 0 0))
   )
-  (wire (pts (xy 36.83 34.29) (xy 36.83 38.1))
-    (stroke (width 0) (type default) (color 0 0 0 0))
-  )
   (wire (pts (xy 135.89 81.28) (xy 139.7 81.28))
     (stroke (width 0) (type default) (color 0 0 0 0))
@@
   )
   (wire (pts (xy 119.38 125.73) (xy 119.38 140.97))
-    (stroke (width 0) (type default) (color 0 0 0 0))
-  )
-  (wire (pts (xy 36.83 30.48) (xy 36.83 31.75))
     (stroke (width 0) (type default) (color 0 0 0 0))
   )
@@
     )
     (pin "1")
-  )
-  (symbol (lib_id "Device:C_Polarized") (at 45.72 34.29 0) (unit 1)
-    (in_bom yes) (on_board yes)
-    (property "Reference" "C1" (id 0) (at 40.64 33.02 0))
-    (property "Value" "100u" (id 1) (at 40.64 35.56 0))
-    (property "Footprint" "Capacitor_THT:CP_Radial_D5.0mm_P2.50mm" (id 2) (at 46.6852 38.1 0)
-      (effects (font (size 1.27 1.27)) hide)
-    )
-    (property "Datasheet" "~" (id 3) (at 45.72 34.29 0)
-      (effects (font (size 1.27 1.27)) hide)
-    )
-    (pin "1")
-    (pin "2")
   )
   (symbol (lib_id "project_lib:TDA2822") (at 133.35 118.11 0) (unit 2)
@@
       (reference "#PWR0111") (unit 1) (value "GND") (footprint "")
     )
-    (path "/08c4b370-b121-44b3-8e20-cf39dc30f2ae"
-      (reference "C1") (unit 1) (value "100u") (footprint "Capacitor_THT:CP_Radial_D5.0mm_P2.50mm")
-    )
     (path "/f16de308-f84e-4fc5-856b-03192071bc5f"
