File: PCB/Digital Theremin.kicad_pcb (KiCad board)
At the start: 2 copper layers, 100 x 63 mm, 59 parts, among them J1 Conn_01x02_Female, J2 AudioJack3_Dual_Switch, J3 USB_B_Micro, J4 Conn_01x03_Female, SW1 SW_Push, SW2 SW_Push, SW3 SW_SPDT, U1 AP2204K-3.0, U2 TDA2822, U3 NE555P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

Commit message: Set DNF
Parts:
- C15: value 10n -> .1u
- D1, D2, D3: value LED -> DNF
- R1: value 200 -> DNF
- R2, R3, R4: value 220 -> DNF
- RV1: value 10k -> DNF
- SW1, SW2: value SW_Push -> DNF
Changed lines of the file:
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@@
       (effects (font (size 1 1) (thickness 0.15)))
     )
-    (fp_text value "LED" (at 1.27 3.96 90) (layer "F.Fab")
+    (fp_text value "DNF" (at 1.27 3.96 90) (layer "F.Fab")
       (effects (font (size 1 1) (thickness 0.15)))
     )
@@
     (descr "CP, Radial series, Radial, pin pitch=2.50mm, , diameter=5mm, Electrolytic Capacitor")
     (tags "CP Radial series Radial pin pitch 2.50mm  diameter 5mm Electrolytic Capacitor")
+    (property "PN" "ESK107M016AC3AA")
     (property "Sheetfile" "Digital Theremin.kicad_sch")
     (property "Sheetname" "")
@@
       (effects (font (size 1 1) (thickness 0.15)))
     )
-    (fp_text value "220" (at 5.08 2.37) (layer "F.Fab")
+    (fp_text value "DNF" (at 5.08 2.37) (layer "F.Fab")
       (effects (font (size 1 1) (thickness 0.15)))
     )
@@
       (effects (font (size 1 1) (thickness 0.15)))
     )
-    (fp_text value "SW_Push" (at 3.75 6.7) (layer "F.Fab")
+    (fp_text value "DNF" (at 3.75 6.7) (layer "F.Fab")
       (effects (font (size 1 1) (thickness 0.15)))
     )
@@
       (effects (font (size 1 1) (thickness 0.15)))
     )
-    (fp_text value "LED" (at 1.27 3.96 90) (layer "F.Fab")
+    (fp_text value "DNF" (at 1.27 3.96 90) (layer "F.Fab")
       (effects (font (size 1 1) (thickness 0.15)))
     )
@@
       (effects (font (size 1 1) (thickness 0.15)))
     )
-    (fp_text value "220" (at 5.08 2.37) (layer "F.Fab")
+    (fp_text value "DNF" (at 5.08 2.37) (layer "F.Fab")
       (effects (font (size 1 1) (thickness 0.15)))
     )
@@
     (descr "CP, Radial series, Radial, pin pitch=2.50mm, , diameter=5mm, Electrolytic Capacitor")
     (tags "CP Radial series Radial pin pitch 2.50mm  diameter 5mm Electrolytic Capacitor")
+    (property "PN" "860010273011")
     (property "Sheetfile" "Digital Theremin.kicad_sch")
     (property "Sheetname" "")
@@
     (descr "CP, Radial series, Radial, pin pitch=2.50mm, , diameter=5mm, Electrolytic Capacitor")
     (tags "CP Radial series Radial pin pitch 2.50mm  diameter 5mm Electrolytic Capacitor")
+    (property "PN" "ESK107M016AC3AA")
     (property "Sheetfile" "Digital Theremin.kicad_sch")
     (property "Sheetname" "")
@@
       (effects (font (size 1 1) (thickness 0.15)))
     )
-    (fp_text value "200" (at 5.08 2.37) (layer "F.Fab")
+    (fp_text value "DNF" (at 5.08 2.37) (layer "F.Fab")
       (effects (font (size 1 1) (thickness 0.15)))
     )
@@
       (effects (font (size 1 1) (thickness 0.15)))
     )
-    (fp_text value "LED" (at 1.27 3.96 90) (layer "F.Fab")
+    (fp_text value "DNF" (at 1.27 3.96 90) (layer "F.Fab")
       (effects (font (size 1 1) (thickness 0.15)))
     )
@@
       (effects (font (size 1 1) (thickness 0.15)))
     )
-    (fp_text value "10k" (at 0 7.41 90) (layer "F.Fab")
+    (fp_text value "DNF" (at 0 7.41 90) (layer "F.Fab")
       (effects (font (size 1 1) (thickness 0.15)))
     )
@@
       (effects (font (size 1 1) (thickness 0.15)))
     )
-    (fp_text value "10n" (at 1.25 2.5) (layer "F.Fab")
+    (fp_text value ".1u" (at 1.25 2.5) (layer "F.Fab")
       (effects (font (size 1 1) (thickness 0.15)))
     )
@@
     (descr "Through hole straight pin header, 2x05, 1.27mm pitch, double rows")
     (tags "Through hole pin header THT 2x05 1.27mm double row")
+    (property "PN" "20021111-00010T1LF")
     (property "Sheetfile" "digital.kicad_sch")
     (property "Sheetname" "Digital")
@@
       (effects (font (size 1 1) (thickness 0.15)))
     )
-    (fp_text value "220" (at 5.08 2.37) (layer "F.Fab")
+    (fp_text value "DNF" (at 5.08 2.37) (layer "F.Fab")
       (effects (font (size 1 1) (thickness 0.15)))
     )
@@
       (effects (font (size 1 1) (thickness 0.15)))
     )
-    (fp_text value "SW_Push" (at 3.75 6.7) (layer "F.Fab")
-      (effects (font (size 1 1) (thickness 0.15)))
-    )
+    (fp_text value "DNF" (at 3.75 6.7) (layer "F.Fab")
+      (effects (font (size 1 1) (thickness 0.15)))
+    )
