File: PCB/Digital Theremin.kicad_sch (KiCad schematic)
At the start: 42 parts, among them J1 Conn_01x02_Female, J2 AudioJack3_Dual_Switch, J3 USB_B_Micro, J4 Conn_01x03_Female, SW1 SW_Push, SW2 SW_Push, SW3 SW_SPDT, U1 AP2204K-3.0, U2 TDA2822

Commit message: Set DNF
Parts:
- D1, D2, D3: value LED -> DNF
- R1, R2, R3, R4: value 220 -> DNF
- RV1: value 10k -> DNF
- SW1, SW2: value SW_Push -> DNF
Other:
- note added: "Amphenol_10104110"
Changed lines of the file:
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@@
+    (effects (font (size 1.27 1.27)) (justify left bottom))
+  )
+  (text "Amphenol_10104110" (at 88.9 190.5 0)
     (effects (font (size 1.27 1.27)) (justify left bottom))
   )
@@
     (in_bom yes) (on_board yes) (fields_autoplaced)
     (property "Reference" "D2" (id 0) (at 31.4325 139.7 0))
-    (property "Value" "LED" (id 1) (at 31.4325 142.24 0))
+    (property "Value" "DNF" (id 1) (at 31.4325 142.24 0))
     (property "Footprint" "LED_THT:LED_D5.0mm" (id 2) (at 33.02 146.05 0)
       (effects (font (size 1.27 1.27)) hide)
@@
       (effects (font (size 1.27 1.27)) (justify right))
     )
-    (property "Value" "10k" (id 1) (at 39.37 52.0699 0)
+    (property "Value" "DNF" (id 1) (at 39.37 52.0699 0)
       (effects (font (size 1.27 1.27)) (justify right))
     )
@@
     (in_bom yes) (on_board yes) (fields_autoplaced)
     (property "Reference" "SW1" (id 0) (at 33.02 100.33 0))
-    (property "Value" "SW_Push" (id 1) (at 33.02 102.87 0))
+    (property "Value" "DNF" (id 1) (at 33.02 102.87 0))
     (property "Footprint" "Button_Switch_THT:SW_PUSH_6mm" (id 2) (at 33.02 102.87 0)
       (effects (font (size 1.27 1.27)) hide)
@@
     (in_bom yes) (on_board yes) (fields_autoplaced)
     (property "Reference" "R3" (id 0) (at 60.96 139.7 90))
-    (property "Value" "220" (id 1) (at 60.96 142.24 90))
+    (property "Value" "DNF" (id 1) (at 60.96 142.24 90))
     (property "Footprint" "Resistor_THT:R_Axial_DIN0207_L6.3mm_D2.5mm_P10.16mm_Horizontal" (id 2) (at 60.96 147.828 90)
       (effects (font (size 1.27 1.27)) hide)
@@
     (in_bom yes) (on_board yes) (fields_autoplaced)
     (property "Reference" "D3" (id 0) (at 31.4325 157.48 0))
-    (property "Value" "LED" (id 1) (at 31.4325 160.02 0))
+    (property "Value" "DNF" (id 1) (at 31.4325 160.02 0))
     (property "Footprint" "LED_THT:LED_D5.0mm" (id 2) (at 33.02 163.83 0)
       (effects (font (size 1.27 1.27)) hide)
@@
       (effects (font (size 1.27 1.27)) (justify right))
     )
-    (property "Value" "220" (id 1) (at 48.26 40.6399 0)
+    (property "Value" "DNF" (id 1) (at 48.26 40.6399 0)
       (effects (font (size 1.27 1.27)) (justify right))
     )
@@
     (in_bom yes) (on_board yes) (fields_autoplaced)
     (property "Reference" "R4" (id 0) (at 60.96 157.48 90))
-    (property "Value" "220" (id 1) (at 60.96 160.02 90))
+    (property "Value" "DNF" (id 1) (at 60.96 160.02 90))
     (property "Footprint" "Resistor_THT:R_Axial_DIN0207_L6.3mm_D2.5mm_P10.16mm_Horizontal" (id 2) (at 60.96 165.608 90)
       (effects (font (size 1.27 1.27)) hide)
@@
     (in_bom yes) (on_board yes) (fields_autoplaced)
     (property "Reference" "SW2" (id 0) (at 34.29 80.01 0))
-    (property "Value" "SW_Push" (id 1) (at 34.29 82.55 0))
+    (property "Value" "DNF" (id 1) (at 34.29 82.55 0))
     (property "Footprint" "Button_Switch_THT:SW_PUSH_6mm" (id 2) (at 34.29 82.55 0)
       (effects (font (size 1.27 1.27)) hide)
@@
     (in_bom yes) (on_board yes)
     (property "Reference" "D1" (id 0) (at 31.75 121.92 0))
-    (property "Value" "LED" (id 1) (at 31.4325 124.46 0))
+    (property "Value" "DNF" (id 1) (at 31.4325 124.46 0))
     (property "Footprint" "LED_THT:LED_D5.0mm" (id 2) (at 33.02 128.27 0)
       (effects (font (size 1.27 1.27)) hide)
@@
     (in_bom yes) (on_board yes) (fields_autoplaced)
     (property "Reference" "R2" (id 0) (at 60.96 121.92 90))
-    (property "Value" "220" (id 1) (at 60.96 124.46 90))
+    (property "Value" "DNF" (id 1) (at 60.96 124.46 90))
     (property "Footprint" "Resistor_THT:R_Axial_DIN0207_L6.3mm_D2.5mm_P10.16mm_Horizontal" (id 2) (at 60.96 130.048 90)
       (effects (font (size 1.27 1.27)) hide)
@@
     )
     (path "/e6eddaa6-98a5-4d64-9567-cf47a7106bdb"
-      (reference "D1") (unit 1) (value "LED") (footprint "LED_THT:LED_D5.0mm")
+      (reference "D1") (unit 1) (value "DNF") (footprint "LED_THT:LED_D5.0mm")
     )
     (path "/07efeeb9-dd24-4559-bd59-4fa07c46e1be"
-      (reference "D2") (unit 1) (value "LED") (footprint "LED_THT:LED_D5.0mm")
+      (reference "D2") (unit 1) (value "DNF") (footprint "LED_THT:LED_D5.0mm")
     )
     (path "/5cdf0f3f-623c-4f8d-b07a-3592cd8d8754"
-      (reference "D3") (unit 1) (value "LED") (footprint "LED_THT:LED_D5.0mm")
+      (reference "D3") (unit 1) (value "DNF") (footprint "LED_THT:LED_D5.0mm")
     )
     (path "/bf87435d-afab-4b5c-8527-03b62990416e"
@@
     )
     (path "/74792002-d4fe-413e-9baa-acc75935710c"
-      (reference "R1") (unit 1) (value "220") (footprint "Resistor_THT:R_Axial_DIN0207_L6.3mm_D2.5mm_P10.16mm_Horizontal")
+      (reference "R1") (unit 1) (value "DNF") (footprint "Resistor_THT:R_Axial_DIN0207_L6.3mm_D2.5mm_P10.16mm_Horizontal")
     )
     (path "/f0af6990-88da-450d-986d-45d2dcd4e23d"
-      (reference "R2") (unit 1) (value "220") (footprint "Resistor_THT:R_Axial_DIN0207_L6.3mm_D2.5mm_P10.16mm_Horizontal")
+      (reference "R2") (unit 1) (value "DNF") (footprint "Resistor_THT:R_Axial_DIN0207_L6.3mm_D2.5mm_P10.16mm_Horizontal")
     )
     (path "/44b485b0-4dc3-47db-9bbe-603cebbf58cf"
-      (reference "R3") (unit 1) (value "220") (footprint "Resistor_THT:R_Axial_DIN0207_L6.3mm_D2.5mm_P10.16mm_Horizontal")
+      (reference "R3") (unit 1) (value "DNF") (footprint "Resistor_THT:R_Axial_DIN0207_L6.3mm_D2.5mm_P10.16mm_Horizontal")
     )
     (path "/75a608db-252e-4b87-9943-1827242560ec"
-      (reference "R4") (unit 1) (value "220") (footprint "Resistor_THT:R_Axial_DIN0207_L6.3mm_D2.5mm_P10.16mm_Horizontal")
+      (reference "R4") (unit 1) (value "DNF") (footprint "Resistor_THT:R_Axial_DIN0207_L6.3mm_D2.5mm_P10.16mm_Horizontal")
     )
     (path "/4c77cde5-684a-415e-a67a-6740fc4c9f53"
@@
     )
     (path "/2e90ce3b-e517-4e3f-ab96-8852c7b1f4bf"
-      (reference "RV1") (unit 1) (value "10k") (footprint "Connector_PinHeader_2.54mm:PinHeader_1x03_P2.54mm_Vertical")
+      (reference "RV1") (unit 1) (value "DNF") (footprint "Connector_PinHeader_2.54mm:PinHeader_1x03_P2.54mm_Vertical")
     )
     (path "/5bf1c4bd-8530-4bc1-8161-1bb532ee9a61"
@@
     )
     (path "/43d7322f-dfb7-4a28-af3b-3eb60d54024c"
-      (reference "SW1") (unit 1) (value "SW_Push") (footprint "Button_Switch_THT:SW_PUSH_6mm")
+      (reference "SW1") (unit 1) (value "DNF") (footprint "Button_Switch_THT:SW_PUSH_6mm")
     )
     (path "/bb4303f1-f627-41a5-8056-3405f923db5e"
-      (reference "SW2") (unit 1) (value "SW_Push") (footprint "Button_Switch_THT:SW_PUSH_6mm")
+      (reference "SW2") (unit 1) (value "DNF") (footprint "Button_Switch_THT:SW_PUSH_6mm")
     )
     (path "/2a39c492-a005-4a5d-95e6-6732324d6eb6"

Commit message: Add how-to
Other:
- note added: "To Fit Case: 1591XXSTBU, 1591XXSSBK, or 1591XXSSFLBK"
- note removed: "To Fit Case: 1591XXSTBU"
